Commit message: add two cameras d435 to urdf

File: rbrobout_description/robots/rbrobout.urdf.xacro (robot description, xacro)
@@ -53,4 +53,10 @@
 			<origin xyz="-0.8 -0.366 -0.06" rpy="0 0 ${-3/4*PI}"/>
 		</xacro:sensor_sick_microscan3>
+		<xacro:sensor_intel_d435 prefix="$(arg prefix)front_rgbd_camera" parent="$(arg prefix)base_link" prefix_topic="front_rgbd_camera">
+      		<origin xyz="0.835 0  0.1555" rpy="0 0 0"/>
+    	</xacro:sensor_intel_d435>
+    		<xacro:sensor_intel_d435 prefix="$(arg prefix)rear_rgbd_camera" parent="$(arg prefix)base_link" prefix_topic="rear_rgbd_camera">
+      		<origin xyz="-0.835 0  0.1555" rpy="0 ${PI} 0"/>
+    	</xacro:sensor_intel_d435>
 		<!-- magnetic sensors  -->
 		<!--xacro:sick_mls prefix="$(arg prefix)left_mls" parent="$(arg prefix)base_link">
